Commit message: Add gripper components to URDF and update SRDF for MoveIt2 integration

File: igus_rebel_description/urdf/igus_rebel2.urdf (robot description, URDF)
Before this commit: robot igus_rebel, 12 links, 11 joints
Links:
- added link gripper_base; collision mesh filename=file://$(find igus_rebel_description)/meshes/gripper_base.s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 scale=0.001 0.001 0.001; visual mesh filename=file://$(find igus_rebel_description)/meshes/gripper_base.s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 scale=0.001 0.001 0.001
- added link gripper_leftfinger; collision mesh filename=file://$(find igus_rebel_description)/meshes/finger_left.stl scale=0.001 0.001 0.001; visual mesh filename=file://$(find igus_rebel_description)/meshes/finger_left.stl scale=0.001 0.001 0.001
- added link gripper_rightfinger; collision mesh filename=file://$(find igus_rebel_description)/meshes/finger_right.s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 scale=0.001 0.001 0.001; visual mesh filename=file://$(find igus_rebel_description)/meshes/finger_right.s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 scale=0.001 0.001 0.001
Joints:
- added joint gripper_leftfinger_joint: type fixed, parent gripper_base, child gripper_leftfinger, origin xyz=0.0955 0 0.01169 rpy=0 0 0
- added joint gripper_link6_joint: type fixed, parent link6, child gripper_base, origin xyz=0 0 0 rpy=0 0 0.0
- added joint gripper_rightfinger_joint: type fixed, parent gripper_base, child gripper_rightfinger, origin xyz=-0.0955 0 0.01169 rpy=0 0 0
